File: Proyecto_ArgibayManuel_YangAlex/Proyecto_ArgibayManuel_YangAlex.kicad_sch (KiCad schematic)
At the start: 38 parts, among them IC1 LM1117, J2 Conn_01x04, J3 Conn_01x06, J4 Conn_01x04, SW1 SW_Push, SW2 SW_Push, SW3 SW_Push, SW4 SW_Push, U1 PIC18F258-I_SO, U10 LT1716IS5TRMPBF, U6 MCP2551-I-P, U9 LT1716IS5TRMPBF, X1 DB9, X2 DB9, Y1 Crystal

Commit message: Ordenar esquematico
Parts:
- removed C10, C11: 500pF, symbol Device:C
- removed C4, C6, C8: 100nF, symbol Device:C
- removed C5, C7: 1uF, symbol Device:C_Polarized_US
- removed D3: 1N4002, Diode_THT:D_DO-41_SOD81_P10.16mm_Horizontal, symbol Diode:1N4002
- removed D4: BZV55C6V2, Diode_SMD:D_MiniMELF, symbol Diode:BZV55C6V2
- removed IC1: LM1117, symbol LM1117:LM1117
- removed R4, R5: 1k, symbol Device:R
- removed R6: 60, symbol Device:R
- removed U6: MCP2551-I-P, Package_DIP:DIP-8_W7.62mm, symbol Interface_CAN_LIN:MCP2551-I-P
- removed X1, X2: DB9, DB9:DB9, symbol DB9:DB9
Connections:
- no-connect marks 11 -> 8
Other:
- added sheet Buses (Buses.kicad_sch)
- added sheet Regulador de Tension (Regulador de tension.kicad_sch)
- note added: "Botonera"
- note added: "Buses"
- note added: "Motores"
- note added: "Regulador de Tension"
- note removed: "Conector DB-9"
- note removed: "MCP2551"
- note removed: "Puentes H"
- note removed: "Regulador de Tensión LM1117"
- moved on the sheet: C1, C2, C3, C9, J2, J3, J4, R10, R11, R12, R3, R7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

Commit message: footprint
Parts:
- added U7: HDC2010YPAR, HDC2010YPAR:BGA6C100X50P2X3_HDC2010YPAR, symbol HDC2010YPAR:HDC2010YPAR
- C1: renamed from C9; footprint (none) -> Capacitor_SMD:C_0805_2012Metric
- C2: renamed from C1; footprint (none) -> Capacitor_SMD:C_0805_2012Metric
- C3: renamed from C2; footprint (none) -> Capacitor_SMD:C_0805_2012Metric
- C4: renamed from C3; footprint (none) -> Capacitor_SMD:C_0805_2012Metric
- J1: renamed from J4; footprint (none) -> Connector_PinHeader_2.54mm:PinHeader_1x04_P2.54mm_Vertical
- J2: footprint (none) -> Connector_PinHeader_2.54mm:PinHeader_1x04_P2.54mm_Vertical
- J3: footprint (none) -> TerminalBlock_Phoenix:TerminalBlock_Phoenix_MKDS-1,5-6_1x06_P5.00mm_Horizontal
- R1: renamed from R12; footprint (none) -> Resistor_THT:R_Axial_DIN0204_L3.6mm_D1.6mm_P1.90mm_Vertical
- R2: renamed from R11; footprint (none) -> Resistor_THT:R_Axial_DIN0204_L3.6mm_D1.6mm_P1.90mm_Vertical
- R3: footprint (none) -> Resistor_THT:R_Axial_DIN0204_L3.6mm_D1.6mm_P1.90mm_Vertical
- R4: renamed from R9; footprint (none) -> Resistor_THT:R_Axial_DIN0204_L3.6mm_D1.6mm_P1.90mm_Vertical
- R5: renamed from R7; footprint (none) -> Resistor_THT:R_Axial_DIN0204_L3.6mm_D1.6mm_P1.90mm_Vertical
- R6: renamed from R10; footprint (none) -> Resistor_THT:R_Axial_DIN0204_L3.6mm_D1.6mm_P1.90mm_Vertical
- R7: renamed from R8; footprint (none) -> Resistor_THT:R_Axial_DIN0204_L3.6mm_D1.6mm_P1.90mm_Vertical
- SW1: renamed from SW2; footprint (none) -> Button_Switch_SMD:SW_Push_1P1T_NO_CK_KMR2
- SW2: renamed from SW3; footprint (none) -> Button_Switch_SMD:SW_Push_1P1T_NO_CK_KMR2
- SW3: renamed from SW4; footprint (none) -> Button_Switch_SMD:SW_Push_1P1T_NO_CK_KMR2
- SW4: renamed from SW1; footprint (none) -> Button_Switch_SMD:SW_Push_1P1T_NO_CK_KMR2
- Y1: footprint (none) -> Crystal:Crystal_HC49-U_Vertical
- renumbered U10 to U2, U9 to U3
Connections:
- net GND: now also U7.C1 (GND)
Other:
- note added: "Sensor Digital"

Commit message: empezando a añadir el sensor(aun no esta terminado)
Parts:
- removed J1: Conn_01x04, Connector_PinHeader_2.54mm:PinHeader_1x04_P2.54mm_Vertical, symbol Connector_Generic:Conn_01x04
- added C12, C13, C14: 100nF, Capacitor_SMD:C_0805_2012Metric, symbol Device:C
- added J4: Conn_01x05, symbol Connector_Generic:Conn_01x05
- added U8: TXS0108EPW, Package_SO:TSSOP-20_4.4x6.5mm_P0.65mm, symbol Logic_LevelTranslator:TXS0108EPW
Connections:
- net +12V: now also J4.1 (Pin_1)
- net F_C_Out1: now also J4.3 (Pin_3)
- net F_C_Out2: now also J4.2 (Pin_2)
- net GND: now also C12.2, C13.1, C14.2, J4.5 (Pin_5), U8.11 (GND)
- net VCC: now also C12.1, U8.19 (VCCB), U8.20 (B1)
- net at U7.A1 (VDD): now also U8.1 (A1)
- new net +3.3V: C13.2, C14.1, J4.4 (Pin_4), U8.10 (OE), U8.2 (VCCA)
- no-connect marks 8 -> 22
Other:
- moved on the sheet: J2, J3, R4, R5, R6, R7, U2, U3, U7

Commit message: sensor
Parts:
- J4: footprint (none) -> Connector_PinHeader_2.54mm:PinHeader_1x04_P2.54mm_Vertical
Connections:
- net SCL: now also U7.B2 (SCL)
- net SDA: now also U7.A2 (SDA)
- net RC6: no longer names the net of U1.17 (RC6/TX/CK)
- net RC7: no longer names the net of U1.18 (RC7/RX/DT)
- no-connect marks 22 -> 26
Other:
- moved on the sheet: C12, C13, U7, U8
